File: AD5933.sch (EAGLE design)
At the start: 76 parts, among them U1 ADG1604BRUZ, U10 ADP3303ARZ-3.3, U11 AD5242BRZ1M, U12 AD5245BRJZ100-R2, U2 AD5933YRSZ, U3 AD5242BRZ1M, U4 AD8606ARZ, U5 ADG1604BRUZ, U7 AD8606ARZ, U8 LTC6904MPMS8TRPBF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

Commit message: Add jumper connections to arduino mega
Parts:
- removed AD: 6, pinhead:PINHD-1X6
- removed IOH: 10, pinhead:PINHD-1X10
- removed IOL, POWER: 8, pinhead:PINHD-1X8
Connections:
- net 5V5: now also PCB1.5V, PCB1.IOREF; no longer POWER.2, POWER.5
- net A01: now also PCB1.2; no longer IOL.3
- net A11: now also PCB1.3; no longer IOL.4
- net EN1: now also PCB1.4; no longer IOL.5
- net GND: now also PCB1.GND., PCB1.GND..; no longer POWER.6, POWER.7
- net SCL: now also PCB1.SCL1; no longer IOH.10
- net SDA: now also PCB1.SDA1; no longer IOH.9
- net SEN: now also PCB1.6; no longer IOH.1
Changed lines of the file:
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@@
 <part name="C2" library="rcl" deviceset="C-US" device="C0805" value="0.1u"/>
 <part name="GND11" library="supply1" deviceset="GND" device=""/>
-<part name="POWER" library="pinhead" deviceset="PINHD-1X8" device="" value="8"/>
-<part name="AD" library="pinhead" deviceset="PINHD-1X6" device="" value="6"/>
-<part name="IOH" library="pinhead" deviceset="PINHD-1X10" device="" value="10"/>
-<part name="IOL" library="pinhead" deviceset="PINHD-1X8" device="" value="8"/>
 <part name="GND18" library="supply1" deviceset="GND" device=""/>
 <part name="U10" library="ADI Batch_1" deviceset="ADP3303ARZ-3.3" device=""/>
@@
 <instance part="C2" gate="G$1" x="27.94" y="-45.72"/>
 <instance part="GND11" gate="1" x="27.94" y="-55.88"/>
-<instance part="POWER" gate="A" x="10.16" y="40.64"/>
-<instance part="AD" gate="A" x="10.16" y="15.24" rot="MR180"/>
-<instance part="IOH" gate="A" x="10.16" y="-20.32" rot="MR180"/>
-<instance part="IOL" gate="A" x="10.16" y="-53.34" rot="MR180"/>
-<instance part="GND18" gate="1" x="-15.24" y="27.94"/>
+<instance part="GND18" gate="1" x="5.08" y="20.32" rot="MR0"/>
 <instance part="JP1" gate="G$1" x="10.16" y="66.04"/>
 <instance part="U12" gate="A" x="73.66" y="99.06" rot="MR0"/>
@@
 <instance part="JP2" gate="1" x="111.76" y="86.36"/>
 <instance part="JP3" gate="1" x="157.48" y="71.12"/>
-<instance part="R17" gate="G$1" x="-10.16" y="2.54" rot="R90"/>
-<instance part="R18" gate="G$1" x="-17.78" y="7.62" rot="R90"/>
-<instance part="VDD12" gate="G$1" x="-10.16" y="12.7"/>
-<instance part="VDD13" gate="G$1" x="-17.78" y="17.78"/>
+<instance part="R17" gate="G$1" x="-99.06" y="63.5" rot="R90"/>
+<instance part="R18" gate="G$1" x="-106.68" y="68.58" rot="R90"/>
+<instance part="VDD12" gate="G$1" x="-99.06" y="73.66"/>
+<instance part="VDD13" gate="G$1" x="-106.68" y="78.74"/>
 <instance part="C3" gate="G$1" x="30.48" y="58.42"/>
 <instance part="C4" gate="G$1" x="40.64" y="58.42"/>
@@
 <instance part="P+7" gate="VCC" x="180.34" y="78.74"/>
 <instance part="P+8" gate="VCC" x="299.72" y="73.66"/>
+<instance part="PCB1" gate="G$1" x="-50.8" y="7.62" rot="MR270"/>
 </instances>
 <busses>
@@
 <pinref part="VDD13" gate="G$1" pin="VDD"/>
 <pinref part="R18" gate="G$1" pin="2"/>
-<wire x1="-17.78" y1="15.24" x2="-17.78" y2="12.7" width="0.1524" layer="91"/>
+<wire x1="-106.68" y1="76.2" x2="-106.68" y2="73.66" width="0.1524" layer="91"/>
 </segment>
 <segment>
 <pinref part="VDD12" gate="G$1" pin="VDD"/>
 <pinref part="R17" gate="G$1" pin="2"/>
-<wire x1="-10.16" y1="10.16" x2="-10.16" y2="7.62" width="0.1524" layer="91"/>
+<wire x1="-99.06" y1="71.12" x2="-99.06" y2="68.58" width="0.1524" layer="91"/>
 </segment>
 <segment>
@@
 </segment>
 <segment>
-<pinref part="IOL" gate="A" pin="5"/>
-<wire x1="7.62" y1="-53.34" x2="-7.62" y2="-53.34" width="0.1524" layer="91"/>
-<label x="-5.08" y="-53.34" size="1.778" layer="95"/>
+<label x="-88.9" y="15.24" size="1.778" layer="95"/>
+<pinref part="PCB1" gate="G$1" pin="4"/>
+<wire x1="-78.74" y1="15.24" x2="-96.52" y2="15.24" width="0.1524" layer="91"/>
 </segment>
 </net>
@@
 </segment>
 <segment>
-<pinref part="IOL" gate="A" pin="3"/>
-<wire x1="7.62" y1="-58.42" x2="-7.62" y2="-58.42" width="0.1524" layer="91"/>
-<label x="-5.08" y="-58.42" size="1.778" layer="95"/>
+<label x="-88.9" y="10.16" size="1.778" layer="95"/>
+<wire x1="-78.74" y1="10.16" x2="-96.52" y2="10.16" width="0.1524" layer="91"/>
+<pinref part="PCB1" gate="G$1" pin="2"/>
 </segment>
 </net>
@@
 </segment>
 <segment>
-<pinref part="IOL" gate="A" pin="4"/>
-<wire x1="7.62" y1="-55.88" x2="-7.62" y2="-55.88" width="0.1524" layer="91"/>
-<label x="-5.08" y="-55.88" size="1.778" layer="95"/>
+<wire x1="-78.74" y1="12.7" x2="-96.52" y2="12.7" width="0.1524" layer="91"/>
+<label x="-88.9" y="12.7" size="1.778" layer="95"/>
+<pinref part="PCB1" gate="G$1" pin="3"/>
 </segment>
 </net>
@@
 </segment>
 <segment>
-<pinref part="IOH" gate="A" pin="9"/>
-<wire x1="7.62" y1="-10.16" x2="-17.78" y2="-10.16" width="0.1524" layer="91"/>
-<label x="-5.08" y="-10.16" size="1.778" layer="95"/>
+<label x="-93.98" y="50.8" size="1.778" layer="95"/>
 <pinref part="R18" gate="G$1" pin="1"/>
-<wire x1="-17.78" y1="-10.16" x2="-20.32" y2="-10.16" width="0.1524" layer="91"/>
-<wire x1="-17.78" y1="-10.16" x2="-17.78" y2="2.54" width="0.1524" layer="91"/>
-<junction x="-17.78" y="-10.16"/>
+<wire x1="-78.74" y1="50.8" x2="-106.68" y2="50.8" width="0.1524" layer="91"/>
+<wire x1="-106.68" y1="50.8" x2="-109.22" y2="50.8" width="0.1524" layer="91"/>
+<wire x1="-106.68" y1="50.8" x2="-106.68" y2="63.5" width="0.1524" layer="91"/>
+<junction x="-106.68" y="50.8"/>
+<pinref part="PCB1" gate="G$1" pin="SDA1"/>
 </segment>
 <segment>
@@
 </segment>
 <segment>
-<pinref part="IOH" gate="A" pin="10"/>
-<label x="-5.08" y="-7.62" size="1.778" layer="95"/>
-<wire x1="7.62" y1="-7.62" x2="-10.16" y2="-7.62" width="0.1524" layer="91"/>
-<wire x1="-10.16" y1="-7.62" x2="-25.4" y2="-7.62" width="0.1524" layer="91"/>
+<label x="-93.98" y="53.34" size="1.778" layer="95"/>
+<wire x1="-78.74" y1="53.34" x2="-99.06" y2="53.34" width="0.1524" layer="91"/>
+<wire x1="-99.06" y1="53.34" x2="-114.3" y2="53.34" width="0.1524" layer="91"/>
 <pinref part="R17" gate="G$1" pin="1"/>
-<wire x1="-10.16" y1="-7.62" x2="-10.16" y2="-2.54" width="0.1524" layer="91"/>
-<junction x="-10.16" y="-7.62"/>
+<wire x1="-99.06" y1="53.34" x2="-99.06" y2="58.42" width="0.1524" layer="91"/>
+<junction x="-99.06" y="53.34"/>
+<pinref part="PCB1" gate="G$1" pin="SCL1"/>
 </segment>
 <segment>
@@
 </segment>
 <segment>
-<pinref part="IOH" gate="A" pin="1"/>
-<wire x1="7.62" y1="-30.48" x2="-7.62" y2="-30.48" width="0.1524" layer="91"/>
-<label x="-5.08" y="-30.48" size="1.778" layer="95"/>
+<pinref part="PCB1" gate="G$1" pin="6"/>
+<label x="-88.9" y="20.32" size="1.778" layer="95"/>
+<wire x1="-78.74" y1="20.32" x2="-96.52" y2="20.32" width="0.1524" layer="91"/>
 </segment>
 </net>
 <net name="5V5" class="1">
 <segment>
-<pinref part="POWER" gate="A" pin="2"/>
-<wire x1="7.62" y1="48.26" x2="-5.08" y2="48.26" width="0.1524" layer="91"/>
-<wire x1="-5.08" y1="48.26" x2="-5.08" y2="40.64" width="0.1524" layer="91"/>
-<pinref part="POWER" gate="A" pin="5"/>
-<wire x1="-5.08" y1="40.64" x2="7.62" y2="40.64" width="0.1524" layer="91"/>
-<wire x1="-5.08" y1="48.26" x2="-5.08" y2="55.88" width="0.1524" layer="91"/>
-<junction x="-5.08" y="48.26"/>
-<label x="-10.16" y="50.8" size="1.778" layer="95"/>
+<wire x1="-20.32" y1="40.64" x2="-5.08" y2="40.64" width="0.1524" layer="91"/>
+<wire x1="-5.08" y1="40.64" x2="-5.08" y2="33.02" width="0.1524" layer="91"/>
+<wire x1="-5.08" y1="33.02" x2="-20.32" y2="33.02" width="0.1524" layer="91"/>
+<wire x1="-5.08" y1="40.64" x2="-5.08" y2="48.26" width="0.1524" layer="91"/>
+<junction x="-5.08" y="40.64"/>
+<label x="0" y="43.18" size="1.778" layer="95" rot="MR0"/>
+<pinref part="PCB1" gate="G$1" pin="5V"/>
+<pinref part="PCB1" gate="G$1" pin="IOREF"/>
 </segment>
 </net>
@@
 </segment>
 <segment>
-<pinref part="POWER" gate="A" pin="7"/>
-<wire x1="7.62" y1="35.56" x2="-15.24" y2="35.56" width="0.1524" layer="91"/>
-<wire x1="-15.24" y1="35.56" x2="-15.24" y2="38.1" width="0.1524" layer="91"/>
-<pinref part="POWER" gate="A" pin="6"/>
-<wire x1="-15.24" y1="38.1" x2="7.62" y2="38.1" width="0.1524" layer="91"/>
+<wire x1="-20.32" y1="27.94" x2="5.08" y2="27.94" width="0.1524" layer="91"/>
+<wire x1="5.08" y1="27.94" x2="5.08" y2="30.48" width="0.1524" layer="91"/>
+<wire x1="5.08" y1="30.48" x2="-20.32" y2="30.48" width="0.1524" layer="91"/>
 <pinref part="GND18" gate="1" pin="GND"/>
-<wire x1="-15.24" y1="30.48" x2="-15.24" y2="35.56" width="0.1524" layer="91"/>
-<junction x="-15.24" y="35.56"/>
+<wire x1="5.08" y1="22.86" x2="5.08" y2="27.94" width="0.1524" layer="91"/>
+<junction x="5.08" y="27.94"/>
+<pinref part="PCB1" gate="G$1" pin="GND."/>
+<pinref part="PCB1" gate="G$1" pin="GND.."/>
 </segment>
 <segment>
@@
 </nets>
 </sheet>
-<sheet>
-<plain>
-</plain>
-<instances>
-<instance part="PCB1" gate="G$1" x="68.58" y="50.8"/>
-</instances>
-<busses>
-</busses>
-<nets>
-</nets>
-</sheet>
