File: AD5933.sch (EAGLE design)
At the start: 80 parts, among them U1 ADG1604BRUZ, U10 ADP3303ARZ-3.3, U11 AD5242BRZ1M, U12 AD5245BRJZ100-R2, U2 AD5933YRSZ, U3 AD5242BRZ1M, U4 AD8606ARZ, U5 ADG1604BRUZ, U7 AD8606ARZ, U8 LTC6904MPMS8TRPBF, U9 ADP3303ARZ-3.3, X1 DC21MMX

Commit message: Complete Routing,Semi Automatic
Connections:
- net U7_INB- renamed U7_INA-
Changed lines of the file:
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@@
 <class number="0" name="default" width="0" drill="0.3048">
 </class>
-<class number="1" name="power 5v" width="0.762" drill="0.6096">
+<class number="1" name="power 5v" width="0.508" drill="0.6096">
 </class>
 </classes>
@@
 <part name="GND36" library="supply1" deviceset="AGND" device=""/>
 <part name="GND37" library="supply1" deviceset="AGND" device=""/>
+<part name="GND38" library="supply1" deviceset="AGND" device=""/>
+<part name="GND39" library="supply1" deviceset="GND" device=""/>
 </parts>
 <sheets>
@@
 <instance part="GND36" gate="VR1" x="309.88" y="43.18"/>
 <instance part="GND37" gate="VR1" x="320.04" y="43.18"/>
+<instance part="GND38" gate="VR1" x="111.76" y="0"/>
+<instance part="GND39" gate="1" x="124.46" y="0"/>
 </instances>
 <busses>
@@
 </segment>
 </net>
-<net name="U7_INB-" class="0">
+<net name="U7_INA-" class="0">
 <segment>
 <pinref part="U5" gate="A" pin="D"/>
@@
 </segment>
 </net>
+<net name="STAR" class="1">
+<segment>
+<pinref part="GND38" gate="VR1" pin="AGND"/>
+<wire x1="111.76" y1="5.08" x2="111.76" y2="7.62" width="0.1524" layer="91"/>
+<wire x1="111.76" y1="7.62" x2="124.46" y2="7.62" width="0.1524" layer="91"/>
+<pinref part="GND39" gate="1" pin="GND"/>
+<wire x1="124.46" y1="2.54" x2="124.46" y2="7.62" width="0.1524" layer="91"/>
+<wire x1="111.76" y1="5.08" x2="111.76" y2="2.54" width="0.1524" layer="91"/>
+</segment>
+</net>
